File: PCB-Design/RoboCoreDesign/RoboCore/RoboCore.kicad_sch (KiCad schematic)
At the start: 26 parts, among them J1 SS-52400-002, J2 B2B-PH-SM4-TB, U1 MCP73871

Commit message: made improvements to the PCB
Connections:
- net VBAT: now also U1.14 (V_{BAT}), U1.15 (V_{BAT}), U1.16 (V_{BAT_SENSE})
- net CHARGING: now reaches R5.2 (-), U1.6 (~{PG})
- net CHARGED: now reaches R4.2 (-), U1.8 (STAT1/~{LBO})
- net CHARGING_POWER_GOOD: now reaches R3.2 (-), U1.7 (STAT2)
Changed lines of the file:
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@@
+		)
+	)
+	(label "CHARGING"
+		(at 62.23 146.05 0)
+		(effects
+			(font
+				(size 1.27 1.27)
+			)
+			(justify left bottom)
 		)
 	)
@@
 		)
 	)
-	(label "CHARGING"
-		(at 16.51 156.21 0)
+	(label "CHARGED"
+		(at 62.23 140.97 0)
 		(effects
 			(font
@@
 	(label "+5V_USB"
 		(at 111.76 135.89 0)
-		(effects
-			(font
-				(size 1.27 1.27)
-			)
-			(justify left bottom)
-		)
-	)
-	(label "CHARGING_POWER_GOOD"
-		(at 16.51 125.73 0)
 		(effects
 			(font
@@
 		)
 	)
+	(label "CHARGING_POWER_GOOD"
+		(at 62.23 125.73 0)
+		(effects
+			(font
+				(size 1.27 1.27)
+			)
+			(justify left bottom)
+		)
+	)
 	(label "+5V_USB"
 		(at 16.51 167.64 0)
@@
 		)
 	)
-	(label "CHARGED"
-		(at 16.51 140.97 0)
+	(label "VBAT"
+		(at 68.58 156.21 180)
 		(effects
 			(font
 				(size 1.27 1.27)
 			)
-			(justify left bottom)
+			(justify right bottom)
 		)
 	)

Commit message: made more changes to the board
Parts:
- removed C3: 4.7uf, Capacitor_SMD:C_0805_2012Metric, symbol PCM_Elektuur:C
Changed lines of the file:
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@@
 	)
 	(junction
-		(at 60.96 175.26)
-		(diameter 0)
-		(color 0 0 0 0)
-	)
-	(junction
 		(at 86.36 53.34)
 		(diameter 0)
@@
 	(wire
 		(pts
-			(xy 60.96 175.26) (xy 68.58 175.26)
-		)
-		(stroke
-			(width 0)
-			(type default)
-		)
-	)
-	(wire
-		(pts
 			(xy 137.16 172.72) (xy 137.16 179.07)
 		)
@@
 	(wire
 		(pts
+			(xy 48.26 175.26) (xy 68.58 175.26)
+		)
+		(stroke
+			(width 0)
+			(type default)
+		)
+	)
+	(wire
+		(pts
 			(xy 62.23 156.21) (xy 58.42 156.21)
 		)
@@
 	(wire
 		(pts
-			(xy 60.96 186.69) (xy 60.96 187.96)
-		)
-		(stroke
-			(width 0)
-			(type default)
-		)
-	)
-	(wire
-		(pts
 			(xy 36.83 43.18) (xy 33.02 43.18)
 		)
@@
 	(wire
 		(pts
-			(xy 60.96 175.26) (xy 60.96 176.53)
-		)
-		(stroke
-			(width 0)
-			(type default)
-		)
-	)
-	(wire
-		(pts
 			(xy 27.94 43.18) (xy 33.02 43.18)
 		)
@@
 	(wire
 		(pts
-			(xy 48.26 175.26) (xy 60.96 175.26)
-		)
-		(stroke
-			(width 0)
-			(type default)
-		)
-	)
-	(wire
-		(pts
 			(xy 128.27 179.07) (xy 128.27 187.96)
 		)
@@
 	)
 	(symbol
-		(lib_id "power:GND")
-		(at 60.96 187.96 0)
-		(unit 1)
-		(exclude_from_sim no)
-		(in_bom yes)
-		(on_board yes)
-		(dnp no)
-		(fields_autoplaced yes)
-		(property "Reference" "#PWR09"
-			(at 60.96 194.31 0)
-			(effects
-				(font
-					(size 1.27 1.27)
-				)
-				(hide yes)
-			)
-		)
-		(property "Value" "GND"
-			(at 60.96 193.04 0)
-			(effects
-				(font
-					(size 1.27 1.27)
-				)
-			)
-		)
-		(property "Footprint" ""
-			(at 60.96 187.96 0)
-			(effects
-				(font
-					(size 1.27 1.27)
-				)
-				(hide yes)
-			)
-		)
-		(property "Datasheet" ""
-			(at 60.96 187.96 0)
-			(effects
-				(font
-					(size 1.27 1.27)
-				)
-				(hide yes)
-			)
-		)
-		(property "Description" "Power symbol creates a global label with name \"GND\" , ground"
-			(at 60.96 187.96 0)
-			(effects
-				(font
-					(size 1.27 1.27)
-				)
-				(hide yes)
-			)
-		)
-		(pin "1"
-		)
-		(instances
-			(project "RoboCore"
-				(path "/4fad5ee2-8ab9-4697-9a8f-c6efe4c71bb3"
-					(reference "#PWR09")
-					(unit 1)
-				)
-			)
-		)
-	)
-	(symbol
 		(lib_id "PCM_Elektuur:C")
 		(at 86.36 64.77 0)
@@
 					(unit 1)
 				)
-			)
-		)
-	)
-	(symbol
-		(lib_id "PCM_Elektuur:C")
-		(at 60.96 181.61 180)
-		(unit 1)
-		(exclude_from_sim no)
-		(in_bom yes)
-		(on_board yes)
-		(dnp no)
-		(fields_autoplaced yes)
-		(property "Reference" "C3"
-			(at 64.77 180.3399 0)
-			(effects
-				(font
-					(size 1.27 1.27)
-				)
-				(justify right)
-			)
-		)
-		(property "Value" "4.7uf"
-			(at 64.77 182.8799 0)
-			(effects
-				(font
-					(size 1.27 1.27)
-				)
-				(justify right)
-			)
-		)
-		(property "Footprint" "Capacitor_SMD:C_0805_2012Metric"
-			(at 60.96 181.61 0)
-			(effects
-				(font
-					(size 1.27 1.27)
-				)
-				(hide yes)
-			)
-		)
-		(property "Datasheet" ""
-			(at 60.96 181.61 0)
-			(effects
-				(font
-					(size 1.27 1.27)
-				)
-				(hide yes)
-			)
-		)
-		(property "Description" "capacitor, non-polarized/bipolar"
-			(at 60.96 181.61 0)
-			(effects
-				(font
-					(size 1.27 1.27)
-				)
-				(hide yes)
-			)
-		)
-		(property "Indicator" "+"
-			(at 62.23 184.785 0)
-			(effects
-				(font
-					(size 1.27 1.27)
-				)
-				(hide yes)
-			)
-		)
-		(property "Rating" "V"
-			(at 61.595 178.435 0)
-			(effects
-				(font
-					(size 1.27 1.27)
-				)
-				(justify right)
-				(hide yes)
-			)
-		)
-		(pin "1"
-		)
-		(pin "2"
-		)
-		(instances
-			(project "RoboCore"
-				(path "/4fad5ee2-8ab9-4697-9a8f-c6efe4c71bb3"
-					(reference "C3")
-					(unit 1)
-				)
