File: PCB-Design/RoboCoreDesign/RoboCore/RoboCore.kicad_sch (KiCad schematic)
At the start: 25 parts, among them J1 SS-52400-002, J2 B2B-PH-SM4-TB, U1 MCP73871

Commit message: made imprvement to the board and added more visual assets of the project
Parts:
- R1, R2: value 5.1k1 -> 5.1k
Connections:
- net VBAT renamed +BATT
Changed lines of the file:
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@@
 			)
 		)
-		(property "Value" "5.1k1"
+		(property "Value" "5.1k"
 			(at 53.34 27.94 90)
 			(effects
@@
 			)
 		)
-		(property "Value" "5.1k1"
+		(property "Value" "5.1k"
 			(at 19.558 75.184 0)
 			(effects
@@
 	)
 	(embedded_fonts no)
+	(wire
+		(pts
+			(xy 180.34 104.14) (xy 180.34 107.95)
+		)
+		(stroke
+			(width 0)
+			(type default)
+		)
+	)
+	(symbol
+		(lib_id "power:+BATT")
+		(at 180.34 107.95 180)
+		(unit 1)
+		(exclude_from_sim no)
+		(in_bom yes)
+		(on_board yes)
+		(dnp no)
+		(fields_autoplaced yes)
+		(property "Reference" "#PWR0102"
+			(at 180.34 111.76 0)
+			(effects
+				(font
+					(size 1.27 1.27)
+				)
+				(hide yes)
+			)
+		)
+		(property "Value" "+BATT"
+			(at 180.34 112.014 0)
+			(effects
+				(font
+					(size 1.27 1.27)
+				)
+			)
+		)
+		(property "Footprint" ""
+			(at 180.34 107.95 0)
+			(effects
+				(font
+					(size 1.27 1.27)
+				)
+				(hide yes)
+			)
+		)
+		(property "Datasheet" ""
+			(at 180.34 107.95 0)
+			(effects
+				(font
+					(size 1.27 1.27)
+				)
+				(hide yes)
+			)
+		)
+		(property "Description" "Power symbol creates a global label with name \"+BATT\""
+			(at 180.34 107.95 0)
+			(effects
+				(font
+					(size 1.27 1.27)
+				)
+				(hide yes)
+			)
+		)
+		(pin "1"
+		)
+		(instances
+			(project "RoboCore"
+				(path "/4fad5ee2-8ab9-4697-9a8f-c6efe4c71bb3"
+					(reference "#PWR0102")
+					(unit 1)
+				)
+			)
+		)
+	)
 )
