File: PCB-Design/RoboCoreDesign/RoboCore/RoboCore.kicad_pcb (KiCad board)
At the start: 4 copper layers, 68 x 60 mm, 81 parts, among them IC1 DRV8245SQRXZRQ1, IC2 DRV8245SQRXZRQ1, J1 SS-52400-002, J2 B2B-PH-SM4-TB, Q1 BC817, Q2 BC817, U1 MCP73871, U2 CP2102N-Axx-xQFN20, U3 USBLC6-2SC6, U4 ESP32-C3-WROOM-02-H4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

Commit message: Refactor code structure for improved readability and maintainability
Parts:
- moved R28 11.7 mm to (149.4, 114.5)
- moved C1 11.5 mm to (154.2, 125.1)
- moved C2 9.54 mm to (157.6, 116.3), turned to 180 degrees
- moved F2 8.54 mm to (157.0, 120.7), turned to 0 degrees
- moved U3 6.22 mm to (149.0, 122.8), turned to -90 degrees
- moved C18 5.48 mm to (184.9, 125.3), turned to -90 degrees
- moved C19 5.48 mm to (181.5, 125.3)
- moved IC1 0.93 mm to (189.5, 123.0)
- moved IC2 0.93 mm to (177.0, 123.0)
- moved R6 0.84 mm to (169.6, 125.7)
- moved R8 0.84 mm to (164.5, 125.7)
- moved R7 0.84 mm to (167.0, 125.7)
- moved R9 0.84 mm to (161.7, 125.7)
- moved R26 0.53 mm to (188.0, 116.2)
Routing:
- net /+5V_USB: vias 0 -> 3
- added copper zone on In1.Cu, net +3.3V
- added copper zone on In1.Cu, net +BATT
- added copper zone on F.Cu, net /+5V_USB
- added copper zone on In1.Cu, net /+5V_USB
- added copper zone on In1.Cu, net /VBUS

Commit message: made improvements to the PCB
Parts:
- J3: renamed from Motor A
- J4: renamed from Motor B
- moved R28 23.0 mm to (171.8, 109.1)
- moved C2 19.7 mm to (157.8, 135.9), turned to 0 degrees
- moved C3 19.2 mm to (157.1, 116.6)
- moved R13 9.62 mm to (163.2, 107.2), turned to 90 degrees
- moved C10 9.50 mm to (156.6, 107.4)
- moved R6 7.80 mm to (161.8, 125.9)
- moved U2 7.57 mm to (151.8, 108.4), turned to 90 degrees
- moved C9 7.06 mm to (159.5, 106.1)
- moved C4 6.01 mm to (141.6, 122.5), turned to 180 degrees
- moved C14 5.34 mm to (176.1, 92.8), turned to 90 degrees
- moved Q2 5.24 mm to (151.0, 93.0)
- moved Q1 4.80 mm to (151.0, 98.0)
- moved R7 2.84 mm to (169.8, 125.9)
- moved R8 2.84 mm to (167.3, 125.9)
- moved R9 2.84 mm to (164.5, 125.9)
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- renumbered PWB to LED4, TX to LED5, RX to LED6, RESET to SW1, BOOT to SW2, FLASH to U6
Connections:
- net Net-(R3--) renamed /CHARGING_POWER_GOOD
- net Net-(R4--) renamed /CHARGED
- net Net-(R5--) renamed /CHARGING
- U1 pad 14: Net-(U1-V_{BAT_SENSE}) -> /VBAT
- U1 pad 15: Net-(U1-V_{BAT_SENSE}) -> /VBAT
- U1 pad 16: Net-(U1-V_{BAT_SENSE}) -> /VBAT
Routing:
- net GND: track 0.00 -> 153.7 mm, vias 0 -> 62
- net +3.3V: track 0.00 -> 79.5 mm, vias 0 -> 26
- net /ESP32_BOARD_CONNECTION/nFAULT_A: track 0.00 -> 65.7 mm, vias 0 -> 2
- net /ESP32_BOARD_CONNECTION/BOOT: track 0.00 -> 53.9 mm, vias 0 -> 2
- net /ESP32_BOARD_CONNECTION/I2C_SDA: track 0.00 -> 53.6 mm, vias 0 -> 2
- net /ESP32_BOARD_CONNECTION/DIR_B: track 0.00 -> 53.3 mm, vias 0 -> 2
- net /ESP32_BOARD_CONNECTION/nFAULT_B: track 0.00 -> 47.5 mm, vias 0 -> 2
- net /ESP32_BOARD_CONNECTION/EN: track 0.00 -> 44.1 mm, vias 0 -> 2
- net /ESP32_BOARD_CONNECTION/RX_TX: track 0.00 -> 37.6 mm, vias 0 -> 4
- net /ESP32_BOARD_CONNECTION/TX_RX: track 0.00 -> 37.3 mm, vias 0 -> 2
- net Net-(C8--): track 0.00 -> 34.0 mm, vias 0 -> 4
- net +5V: track 0.00 -> 33.6 mm
- net /ESP32_BOARD_CONNECTION/SPI_MOSI: track 0.00 -> 29.0 mm
- net /VBAT: track 0.00 -> 28.5 mm
- net Net-(R15--): track 0.00 -> 26.9 mm, vias 0 -> 2
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- added copper zone on F.Cu, net +3.3V
- added copper zone on F.Cu, net +5V
- added copper zone on F.Cu, net /VBAT
- added copper zone on F.Cu, net /VBUS
- added copper zone on F.Cu, net GND
Other:
- outline, holes or cut-outs redrawn

Commit message: made more changes to the board
Parts:
- removed C3: 4.7uf, Capacitor_SMD:C_0805_2012Metric
Routing:
- net /ESP32_BOARD_CONNECTION/DIR_A: track 0.00 -> 65.2 mm, vias 0 -> 2
- net /ESP32_BOARD_CONNECTION/PWM_A: track 0.00 -> 64.4 mm
- net /ESP32_BOARD_CONNECTION/PWM_B: track 24.0 -> 62.3 mm, vias 4 -> 6
- net Net-(IC2-NSLEEP): track 0.00 -> 13.1 mm, vias 0 -> 2
- net Net-(IC1-NSLEEP): track 0.00 -> 10.1 mm, vias 0 -> 2
- net Net-(IC1-SR): track 16.5 -> 13.5 mm
- net GND: track 153.7 -> 152.3 mm
- net Net-(IC1-DRVOFF): track 15.4 -> 16.5 mm
- net +5V: vias 0 -> 1

Commit message: a few changes to the board's layout
Parts:
- moved C10 33.5 mm to (127.8, 90.1)
- moved C18 33.5 mm to (156.2, 108.0)
- moved C5 33.5 mm to (112.8, 108.1)
- moved F2 33.5 mm to (128.3, 103.3)
- moved H3 33.5 mm to (105.3, 118.3)
- moved J3 33.5 mm to (159.3, 114.0)
- moved R15 33.5 mm to (140.7, 90.6)
- moved R2 33.5 mm to (111.3, 119.0)
- moved R29 33.5 mm to (146.3, 90.5)
- moved U1 33.5 mm to (129.4, 114.2)
- moved C13 33.5 mm to (162.7, 86.3)
- moved C15 33.5 mm to (163.9, 76.5)
- moved C4 33.5 mm to (112.8, 105.2)
- moved C8 33.5 mm to (126.3, 96.9)
- moved LED1 33.5 mm to (131.9, 96.2)
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- renumbered SW2 to BOOT, LED4 to PWD, SW1 to RESET, LED5 to RX, LED6 to TX
Routing:
- net GND: track 152.3 -> 162.2 mm, vias 62 -> 302
- net /ESP32_BOARD_CONNECTION/BOOT: track 53.9 -> 55.6 mm
- net /ESP32_BOARD_CONNECTION/RX_TX: track 37.6 -> 39.3 mm
- net /ESP32_BOARD_CONNECTION/I2C_SDA: track 53.4 -> 52.7 mm
- net +BATT: vias 4 -> 0
- added copper zone on F.Cu, net +BATT
- removed copper zone on In1.Cu, net +BATT

Commit message: made more changes
Parts:
- CHARGE PWR: renamed from LED3
- MOTOR 1: renamed from J4
- MOTOR 2: renamed from J3
- renumbered LED2 to CHARGED, LED1 to CHARGING
Other:
- board text added: "CHARGER"
- board text added: "DRIVER"
- board text added: "ESP32"
- board text added: "FLASH MEMORY"
- board text added: "MOTOR"
- board text added: "MPU 6050"
- board text added: "REGULATOR"
- board text added: "USB"

Commit message: made more changes
Routing:
- added copper zone on F.Cu, net Net-(IC2-NSLEEP)
Other:
- board text added: "DRIVERS"
- board text removed: "DRIVER"
Changed lines of the file:
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@@
 			)
 		)
+		(model "${MODELS}/LTST-C171KRKT.stp"
+			(offset
+				(xyz 0 0 0)
+			)
+			(scale
+				(xyz 1 1 1)
+			)
+			(rotate
+				(xyz -90 -0 -0)
+			)
+		)
 	)
 	(footprint "Resistor_SMD:R_0805_2012Metric"
@@
 			)
 		)
+		(model "${MODELS}/T491A475K010AT.step"
+			(offset
+				(xyz 0 0 0)
+			)
+			(scale
+				(xyz 1 1 1)
+			)
+			(rotate
+				(xyz -90 -0 -0)
+			)
+		)
 	)
 	(footprint "Resistor_SMD:R_0805_2012Metric"
@@
 			)
 		)
+		(model "${MODELS}/LTST-C171KRKT.stp"
+			(offset
+				(xyz 0 0 0)
+			)
+			(scale
+				(xyz 1 1 1)
+			)
+			(rotate
+				(xyz -90 -0 -0)
+			)
+		)
 	)
 	(footprint "Resistor_SMD:R_0805_2012Metric"
@@
 		(tags "Capacitor Polarised")
 		(property "Reference" "C11"
-			(at -2.06 3.813 180)
+			(at -2.06 3.813 0)
 			(layer "F.SilkS")
 			(effects
@@
 			)
 		)
+		(model "${MODELS}/T491A475K010AT.step"
+			(offset
+				(xyz 0 0 0)
+			)
+			(scale
+				(xyz 1 1 1)
+			)
+			(rotate
+				(xyz -90 -0 -0)
+			)
+		)
 	)
 	(footprint "RoboCoreFootPrints1:T491A"
@@
 			)
 		)
+		(model "${MODELS}/T491A475K010AT.step"
+			(offset
+				(xyz 0 0 0)
+			)
+			(scale
+				(xyz 1 1 1)
+			)
+			(rotate
+				(xyz -90 -0 -0)
+			)
+		)
 	)
 	(footprint "Resistor_SMD:R_0805_2012Metric"
@@
 			)
 		)
+		(model "${MODELS}/LTST-C171KRKT.stp"
+			(offset
+				(xyz 0 0 0)
+			)
+			(scale
+				(xyz 1 1 1)
+			)
+			(rotate
+				(xyz -90 -0 -0)
+			)
+		)
 	)
 	(footprint "RoboCoreFootPrints1:LEDC2012X120N"
@@
 			)
 		)
+		(model "${MODELS}/LTST-C171KRKT.stp"
+			(offset
+				(xyz 0 0 0)
+			)
+			(scale
+				(xyz 1 1 1)
+			)
+			(rotate
+				(xyz -90 -0 -0)
+			)
+		)
 	)
 	(footprint "Resistor_SMD:R_0805_2012Metric"
@@
 			)
 		)
+		(model "${MODELS}/LTST-C171KRKT.stp"
+			(offset
+				(xyz 0 0 0)
+			)
+			(scale
+				(xyz 1 1 1)
+			)
+			(rotate
+				(xyz -90 -0 -0)
+			)
+		)
 	)
 	(footprint "Resistor_SMD:R_0805_2012Metric"
@@
 			)
 		)
+		(model "${MODELS}/LTST-C171KRKT.stp"
+			(offset
+				(xyz 0 0 0)
+			)
+			(scale
+				(xyz 1 1 1)
+			)
+			(rotate
+				(xyz -90 -0 -0)
+			)
+		)
 	)
 	(footprint "RoboCoreFootPrints1:JST_B2B-PH-SM4-TB"
@@
 			)
 		)
+		(model "${MODELS}/T491A475K010AT.step"
+			(offset
+				(xyz 0 0 0)
+			)
+			(scale
+				(xyz 1 1 1)
+			)
+			(rotate
+				(xyz -90 -0 -0)
+			)
+		)
 	)
 	(footprint "Package_TO_SOT_SMD:SOT-23"
@@
 	)
 	(gr_text "MOTOR\n"
-		(at 164.15 106.5 0)
+		(at 151.55 99.5 0)
 		(layer "F.SilkS")
 		(effects
@@
 		)
 	)
-	(gr_text "\nDRIVER\n"
-		(at 164.15 108.15 0)
+	(gr_text "DRIVERS\n\n"
+		(at 151.25 102.7 0)
 		(layer "F.SilkS")
 		(effects
@@
 			)
 		)
+	)
+	(zone
+		(net 21)
+		(net_name "Net-(IC2-NSLEEP)")
+		(layer "F.Cu")
+		(hatch edge 0.5)
+		(priority 14)
+		(connect_pads yes
+			(clearance 0.001)
+		)
+		(min_thickness 0.25)
+		(filled_areas_thickness no)
+		(fill yes
+			(thermal_gap 0.5)
+			(thermal_bridge_width 0.5)
+		)
+		(polygon
+			(pts
+				(xy 147.6 104.15) (xy 147.6 104.65) (xy 142.9 104.65) (xy 142.4 104.15) (xy 142.4 103.55) (xy 142.8 103.15)
+				(xy 143.65 103.15) (xy 144.65 104.15)
+			)
+		)
