File: PCB-Design/RoboCoreDesign/RoboCore/_autosave-RoboCore.kicad_pcb (KiCad board)
At the start: 4 copper layers, 68 x 60 mm, 80 parts, among them IC1 DRV8245SQRXZRQ1, IC2 DRV8245SQRXZRQ1, J1 SS-52400-002, J2 B2B-PH-SM4-TB, J3 MOTOR_A, J4 MOTOR_B, Q1 BC817, Q2 BC817, SW1 RESET, SW2 BOOT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

Commit message: another attempt at correcting the errors but i've yet again failed terribly
Routing:
- net /ESP32_BOARD_CONNECTION/PWM_B: track 61.9 -> 59.8 mm
Changed lines of the file:
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@@
 	)
 	(segment
-		(start 147.85 90.65)
-		(end 147.85 91.4)
+		(start 148.694 93.404531)
+		(end 148.694 103.826998)
+		(width 0.2)
+		(layer "B.Cu")
+		(net 24)
+	)
+	(segment
+		(start 148.95 92.5)
+		(end 148.95 93.148531)
+		(width 0.2)
+		(layer "B.Cu")
+		(net 24)
+	)
+	(segment
+		(start 148.95 93.148531)
+		(end 148.694 93.404531)
 		(width 0.2)
 		(layer "B.Cu")
@@
 	(segment
 		(start 147.85 91.4)
-		(end 148.694 92.244)
+		(end 148.95 92.5)
 		(width 0.2)
 		(layer "B.Cu")
@@
 	)
 	(segment
-		(start 148.694 92.244)
-		(end 148.694 103.826998)
+		(start 147.85 90.65)
+		(end 147.85 91.4)
 		(width 0.2)
 		(layer "B.Cu")
@@
 	)
 	(segment
-		(start 147.55 94.45)
-		(end 147.55 94.95)
+		(start 149.95 97.35)
+		(end 149.1 97.35)
 		(width 0.2)
 		(layer "F.Cu")
@@
 	)
 	(segment
-		(start 147.55 94.95)
-		(end 149.95 97.35)
+		(start 146.4 71.1)
+		(end 145.719 71.781)
 		(width 0.2)
 		(layer "F.Cu")
@@
 	)
 	(segment
-		(start 146.4 71.1)
-		(end 145.719 71.781)
+		(start 149.1 97.35)
+		(end 147.55 95.8)
 		(width 0.2)
 		(layer "F.Cu")
@@
 	)
 	(segment
+		(start 147.55 95.8)
+		(end 147.55 94.9)
+		(width 0.2)
+		(layer "F.Cu")
+		(net 25)
+	)
+	(segment
 		(start 145.719 71.781)
 		(end 144.2745 71.781)
@@
 	)
 	(via
-		(at 147.55 94.45)
+		(at 147.55 94.9)
 		(size 0.6)
 		(drill 0.3)
@@
 	)
 	(segment
-		(start 146.7 82.65)
-		(end 145.4 83.95)
+		(start 160.05 76.85)
+		(end 160.05 72.55)
 		(width 0.2)
 		(layer "B.Cu")
@@
 	)
 	(segment
-		(start 160.05 76.85)
-		(end 160.05 72.55)
+		(start 152.3 81.4)
+		(end 145.4 88.3)
 		(width 0.2)
 		(layer "B.Cu")
@@
 	)
 	(segment
-		(start 145.4 92.25)
-		(end 147.55 94.4)
-		(width 0.2)
-		(layer "B.Cu")
-		(net 25)
-	)
-	(segment
-		(start 147.55 94.4)
-		(end 147.55 94.45)
-		(width 0.2)
-		(layer "B.Cu")
-		(net 25)
-	)
-	(segment
 		(start 154.5 78.7)
 		(end 155.95 77.25)
@@
 	)
 	(segment
-		(start 151.05 82.65)
-		(end 146.7 82.65)
-		(width 0.2)
-		(layer "B.Cu")
-		(net 25)
-	)
-	(segment
 		(start 146.75 70.75)
 		(end 146.4 71.1)
@@
 	)
 	(segment
-		(start 150.3 97.7)
-		(end 150.3 102.45)
+		(start 145.4 92.75)
+		(end 147.55 94.9)
 		(width 0.2)
 		(layer "B.Cu")
@@
 	)
 	(segment
-		(start 158.9 71.4)
-		(end 158.9 71.2)
+		(start 145.4 88.3)
+		(end 145.4 92.75)
 		(width 0.2)
 		(layer "B.Cu")
@@
 	)
 	(segment
-		(start 146.95 70.75)
-		(end 146.75 70.75)
+		(start 150.3 97.7)
+		(end 150.3 102.45)
 		(width 0.2)
 		(layer "B.Cu")
@@
 	)
 	(segment
-		(start 145.4 83.95)
-		(end 145.4 92.25)
+		(start 158.9 71.4)
+		(end 158.9 71.2)
 		(width 0.2)
 		(layer "B.Cu")
@@
 	)
 	(segment
-		(start 152.3 81.4)
-		(end 151.05 82.65)
+		(start 146.95 70.75)
+		(end 146.75 70.75)
 		(width 0.2)
 		(layer "B.Cu")
@@
 	(segment
 		(start 148.3 91.1735)
-		(end 148.3 92.95)
+		(end 148.3 92.949998)
 		(width 0.2)
 		(layer "F.Cu")
@@
 	)
 	(segment
-		(start 148.3 92.95)
-		(end 148.25 93)
-		(width 0.2)
-		(layer "F.Cu")
-		(net 27)
-	)
-	(segment
-		(start 150.05 89.4235)
-		(end 148.3 91.1735)
-		(width 0.2)
-		(layer "F.Cu")
-		(net 27)
-	)
-	(segment
-		(start 148.25 93)
-		(end 148.094 93)
+		(start 148.3 92.949998)
+		(end 148.300002 92.95)
 		(width 0.2)
 		(layer "F.Cu")
@@
 		(net 27)
 	)
+	(segment
+		(start 150.05 89.4235)
+		(end 148.3 91.1735)
+		(width 0.2)
+		(layer "F.Cu")
+		(net 27)
+	)
 	(via
-		(at 148.094 93)
+		(at 148.300002 92.95)
 		(size 0.6)
 		(drill 0.4)
@@
 	)
 	(segment
-		(start 148.094 93)
-		(end 148.294 93.2)
+		(start 148.294 92.956002)
+		(end 148.300002 92.95)
 		(width 0.2)
 		(layer "B.Cu")
@@
 	)
 	(segment
-		(start 148.294 93.2)
+		(start 145.95 101.9)
 		(end 148.294 99.556)
 		(width 0.2)
@@
 	(segment
 		(start 148.294 99.556)
-		(end 145.95 101.9)
+		(end 148.294 92.956002)
 		(width 0.2)
 		(layer "B.Cu")
@@
 		(name "+BATT")
 		(hatch edge 0.5)
-		(priority 17)
+		(priority 6)
 		(connect_pads yes
 			(clearance 0.0001)
