File: PCB-Design/RoboCoreDesign/RoboCore/Buttons.kicad_sch (KiCad schematic)
At the start: 13 parts, among them Q1 BC817, Q2 BC817, SW1 RESET, SW2 BOOT

Commit message: made imprvement to the board and added more visual assets of the project
Parts:
- C21: value 0.uf -> 0.1uf
Changed lines of the file:
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@@
 			)
 		)
-		(property "Value" "0.uf"
+		(property "Value" "0.1uf"
 			(at 166.37 138.4299 0)
 			(effects
