File: PCB-Design/RoboCoreDesign/RoboCore/ESP32_BOARD_CONNECTION.kicad_sch (KiCad schematic)
At the start: 26 parts, among them U2 CP2102N-Axx-xQFN20, U3 USBLC6-2SC6, U4 ESP32-C3-WROOM-02-H4, U5 MPU-6050, U6 W25Q32JVSSIQ

Commit message: made imprvement to the board and added more visual assets of the project
Parts:
- added R33: 10K, Resistor_SMD:R_0805_2012Metric, symbol PCM_Elektuur:R
- C15: value 2.2uf -> 2.2nf
- R16: now not fitted; now left out of the parts list
Connections:
- net +3.3V: now also R13.1 (+), U2.6 (VDD), R33.1 (+)
- net DIR_A: now also R33.2 (-)
- net GND: now also U5.9 (AD0)
- net I2C_SCL: now also U4.8 (IO9)
- net I2C_SDA: no longer U4.8 (IO9)
- net SPI_MISO: now also R16.1 (+), U4.6 (IO7)
- no-connect marks 9 -> 8
