File: PCB-Design/RoboCoreDesign/RoboCore/MotorDriver.kicad_sch (KiCad schematic)
At the start: 16 parts, among them IC1 DRV8245SQRXZRQ1, IC2 DRV8245SQRXZRQ1, J3 MOTOR_A, J4 MOTOR_B

Commit message: made imprvement to the board and added more visual assets of the project
Parts:
- IC1, IC2: value DRV8245SQRXZRQ1 -> DRV8245HQRXZRQ1; Arrow Part Number DRV8245SQRXZRQ1 -> DRV8245HQRXZRQ1; Manufacturer_Part_Number DRV8245SQRXZRQ1 -> DRV8245HQRXZRQ1; Mouser Part Number 595-DRV8245SQRXZRQ1 -> 595-DRV8245HQRXZRQ1; Mouser Price/Stock https://www.mouser.co.uk/ProductDetail/Texas-Instruments/DRV8245SQRXZRQ1?qs=IPgv5n7u5QZV%2FxBh4uiovQ%3D%3D -> https://www.mouser.co.uk/ProductDetail/Texas-Instruments/DRV8245HQRXZRQ1?qs=IPgv5n7u5QZV%2FxBh4uiovQ%3D%3D
Changed lines of the file:
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@@
 			)
 		)
-		(property "Value" "DRV8245SQRXZRQ1"
+		(property "Value" "DRV8245HQRXZRQ1"
 			(at 114.3 133.35 0)
 			(effects
@@
 			)
 		)
-		(property "Manufacturer_Part_Number" "DRV8245SQRXZRQ1"
+		(property "Manufacturer_Part_Number" "DRV8245HQRXZRQ1"
 			(at 127 733.35 0)
 			(effects
@@
 			)
 		)
-		(property "Mouser Part Number" "595-DRV8245SQRXZRQ1"
+		(property "Mouser Part Number" "595-DRV8245HQRXZRQ1"
 			(at 127 833.35 0)
 			(effects
@@
 			)
 		)
-		(property "Mouser Price/Stock" "https://www.mouser.co.uk/ProductDetail/Texas-Instruments/DRV8245SQRXZRQ1?qs=IPgv5n7u5QZV%2FxBh4uiovQ%3D%3D"
+		(property "Mouser Price/Stock" "https://www.mouser.co.uk/ProductDetail/Texas-Instruments/DRV8245HQRXZRQ1?qs=IPgv5n7u5QZV%2FxBh4uiovQ%3D%3D"
 			(at 127 933.35 0)
 			(effects
@@
 			)
 		)
-		(property "Arrow Part Number" "DRV8245SQRXZRQ1"
+		(property "Arrow Part Number" "DRV8245HQRXZRQ1"
 			(at 127 1033.35 0)
 			(effects
@@
 			)
 		)
-		(property "Value" "DRV8245SQRXZRQ1"
+		(property "Value" "DRV8245HQRXZRQ1"
 			(at 120.65 50.8 0)
 			(effects
@@
 			)
 		)
-		(property "Manufacturer_Part_Number" "DRV8245SQRXZRQ1"
+		(property "Manufacturer_Part_Number" "DRV8245HQRXZRQ1"
 			(at 133.35 650.8 0)
 			(effects
@@
 			)
 		)
-		(property "Mouser Part Number" "595-DRV8245SQRXZRQ1"
+		(property "Mouser Part Number" "595-DRV8245HQRXZRQ1"
 			(at 133.35 750.8 0)
 			(effects
@@
 			)
 		)
-		(property "Mouser Price/Stock" "https://www.mouser.co.uk/ProductDetail/Texas-Instruments/DRV8245SQRXZRQ1?qs=IPgv5n7u5QZV%2FxBh4uiovQ%3D%3D"
+		(property "Mouser Price/Stock" "https://www.mouser.co.uk/ProductDetail/Texas-Instruments/DRV8245HQRXZRQ1?qs=IPgv5n7u5QZV%2FxBh4uiovQ%3D%3D"
 			(at 133.35 850.8 0)
 			(effects
@@
 			)
 		)
-		(property "Arrow Part Number" "DRV8245SQRXZRQ1"
+		(property "Arrow Part Number" "DRV8245HQRXZRQ1"
 			(at 133.35 950.8 0)
 			(effects
